Commit message: [modified] gripper pose

File: vs087_with_robotiq_3f_gripper_description/urdf/vs087_with_robotiq_3f_gripper_gazebo.xacro (robot description, xacro)
@@ -238,5 +238,5 @@
   </gazebo>
   <joint name="gripper_joint" type="fixed">
-  <origin xyz="0 0 0.038" rpy="${pi/2} 0 0"/>
+  <origin xyz="0 0 0.038" rpy="${pi/2} 0 ${pi}"/>
   <parent link="J6"/>
   <child link="palm"/>
